Commit message: Movement action working

File: install/roarm_moveit/share/roarm_moveit/config/roarm_description.ros2_control.xacro (robot description, xacro)
@@ -1,40 +1 @@
-<?xml version="1.0"?>
-<robot xmlns:xacro="http://www.ros.org/wiki/xacro">
-    <xacro:macro name="roarm_description_ros2_control" params="name initial_positions_file">
-        <xacro:property name="initial_positions" value="${load_yaml(initial_positions_file)['initial_positions']}"/>
-        <ros2_control name="${name}" type="system">
-            <hardware>
-                <!-- By default, set up controllers for simulation. This won't work on real hardware -->
-                <plugin>mock_components/GenericSystem</plugin>
-            </hardware>
-            <joint name="base_link_to_link1">
-                <command_interface name="position"/>
-                <state_interface name="position">
-                  <param name="initial_value">${initial_positions['base_link_to_link1']}</param>
-                </state_interface>
-                <state_interface name="velocity"/>
-            </joint>
-            <joint name="link1_to_link2">
-                <command_interface name="position"/>
-                <state_interface name="position">
-                  <param name="initial_value">${initial_positions['link1_to_link2']}</param>
-                </state_interface>
-                <state_interface name="velocity"/>
-            </joint>
-            <joint name="link2_to_link3">
-                <command_interface name="position"/>
-                <state_interface name="position">
-                  <param name="initial_value">${initial_positions['link2_to_link3']}</param>
-                </state_interface>
-                <state_interface name="velocity"/>
-            </joint>
-            <joint name="link3_to_gripper_link">
-                <command_interface name="position"/>
-                <state_interface name="position">
-                  <param name="initial_value">${initial_positions['link3_to_gripper_link']}</param>
-                </state_interface>
-                <state_interface name="velocity"/>
-            </joint>
-        </ros2_control>
-    </xacro:macro>
-</robot>
+/home/ws/roarm_ws_em0/src/roarm_main/roarm_moveit/config/roarm_description.ros2_control.xacro

File: install/roarm_moveit/share/roarm_moveit/config/roarm_description.urdf.xacro (robot description, xacro)
@@ -1,9 +1 @@
-<?xml version="1.0"?>
-<robot xmlns:xacro="http://www.ros.org/wiki/xacro" name="roarm_description">
-    <xacro:arg name="initial_positions_file" default="initial_positions.yaml" />
-    <!-- Import roarm_description urdf file -->
-    <xacro:include filename="$(find roarm_description)/urdf/roarm_description.urdf" />
-    <!-- Import control_xacro -->
-    <xacro:include filename="roarm_description.ros2_control.xacro" />
-    <xacro:roarm_description_ros2_control name="FakeSystem" initial_positions_file="$(arg initial_positions_file)"/>
-</robot>
+/home/ws/roarm_ws_em0/src/roarm_main/roarm_moveit/config/roarm_description.urdf.xacro
